Commit message: new data

File: src/cartographer_ros/cartographer_ros/urdf/rplidar.urdf (robot description, URDF)
Before this commit: robot cartographer_backpack_2d, 4 links, 3 joints
Joints:
- joint imu_joint: origin xyz=0.255 0 0 rpy=3.141593 0 0 -> xyz=0 0 0 rpy=0 0 0

Commit message: issue when add imu

File: src/cartographer_ros/cartographer_ros/urdf/rplidar.urdf (robot description, URDF)
Before this commit: robot cartographer_backpack_2d, 4 links, 3 joints
Links:
- removed link odom
Joints:
- removed joint odom_joint
